File: common_emmiter_amplifier/common_emmiter_amplifier.kicad_pcb (KiCad board)
At the start: 2 copper layers, 30.5 x 30.5 mm, 17 parts, among them Q1 2N3904

Commit message: could be final version?
Parts:
- added U1: RH-5000, RH-5000:TEST-TH_BD2.54-P1.4_RED, F.Cu at (130.8, 88.9)
- added U2: RH-5000, RH-5000:TEST-TH_BD2.54-P1.4_RED, F.Cu at (163.8, 88.9)
- added U3: RH-5000, RH-5000:TEST-TH_BD2.54-P1.4_RED, F.Cu at (163.8, 95.2)
- added U4: RH-5000, RH-5000:TEST-TH_BD2.54-P1.4_RED, F.Cu at (130.8, 95.2)
- TP1, TP2, TP3, TP4, TP5, TP6: footprint TestPoint:TestPoint_THTPad_3.0x3.0mm_Drill1.5mm -> TestPoint:TestPoint_THTPad_D3.0mm_Drill1.5mm
- moved TP2 0.90 mm to (159.4, 104.8)
- moved TP3 0.90 mm to (159.4, 80.6)
- moved TP4 0.90 mm to (135.3, 104.8)
- moved TP6 0.90 mm to (135.3, 80.6)
- moved TP1 0.63 mm to (135.3, 92.7)
- moved TP5 0.63 mm to (159.4, 89.4)
- moved kibuzzard-66C691BF 0.63 mm to (159.4, 96.8)
Routing:
- net GND: track 26.5 -> 53.7 mm
- net Net-(C1-Pad2): track 3.81 -> 12.7 mm
- net Net-(Q1-C): track 14.0 -> 18.6 mm
Other:
- board size 30.5 x 30.5 mm -> 38.1 x 30.5 mm
