File: common_emmiter_amplifier/common_emmiter_amplifier.kicad_sch (KiCad schematic)
At the start: 13 parts, among them Q1 2N3904

Commit message: could be final version?
Parts:
- added U1, U2, U3, U4: RH-5000, RH-5000:TEST-TH_BD2.54-P1.4_RED, symbol RH-5000:RH-5000
- TP1, TP2, TP3, TP4, TP5, TP6: footprint TestPoint:TestPoint_THTPad_3.0x3.0mm_Drill1.5mm -> TestPoint:TestPoint_THTPad_D3.0mm_Drill1.5mm
Connections:
- net GND: now also U3.1, U4.1
- net at Q1.3 (C), R3.2, TP5.1: now also U2.1
- net at C1.2, TP1.1: now also U1.1
